File: FloppyShield/Floppy Shield.sch (EAGLE design)
At the start: 13 parts

Commit message: Shield now works with "crossover" floppy cables  (grounded DRIVE A SELECT)
Connections:
- net GND: now also FLP1-14.S, FLP2-14.S, FLP3-14.S, FLP4-14.S
Changed lines of the file:
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@@
 <pinref part="GND8" gate="1" pin="GND"/>
 <wire x1="175.26" y1="60.96" x2="177.8" y2="60.96" width="0.1524" layer="91"/>
+<pinref part="FLP1" gate="-14" pin="S"/>
+<wire x1="177.8" y1="60.96" x2="177.8" y2="55.88" width="0.1524" layer="91"/>
+<junction x="177.8" y="60.96"/>
 </segment>
 <segment>
@@
 <pinref part="GND9" gate="1" pin="GND"/>
 <wire x1="220.98" y1="60.96" x2="223.52" y2="60.96" width="0.1524" layer="91"/>
+<pinref part="FLP2" gate="-14" pin="S"/>
+<wire x1="223.52" y1="60.96" x2="223.52" y2="55.88" width="0.1524" layer="91"/>
+<junction x="223.52" y="60.96"/>
 </segment>
 <segment>
@@
 <pinref part="GND10" gate="1" pin="GND"/>
 <wire x1="266.7" y1="60.96" x2="269.24" y2="60.96" width="0.1524" layer="91"/>
+<pinref part="FLP3" gate="-14" pin="S"/>
+<wire x1="269.24" y1="60.96" x2="269.24" y2="55.88" width="0.1524" layer="91"/>
+<junction x="269.24" y="60.96"/>
 </segment>
 <segment>
@@
 <pinref part="GND11" gate="1" pin="GND"/>
 <wire x1="312.42" y1="60.96" x2="314.96" y2="60.96" width="0.1524" layer="91"/>
+<pinref part="FLP4" gate="-14" pin="S"/>
+<wire x1="314.96" y1="60.96" x2="314.96" y2="55.88" width="0.1524" layer="91"/>
+<junction x="314.96" y="60.96"/>
 </segment>
 <segment>
